File: mmp.kicad_sch (KiCad schematic)
At the start: 26 parts, among them J2 Conn_01x06_Socket, SW1 SW_Push, SW10 SW_Push, SW11 SW_Push, SW12 SW_Push, SW2 SW_Push, SW3 SW_Push, SW4 SW_Push, SW5 SW_Push, SW6 SW_Push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

Commit message: Initial pcb layout
Parts:
- D1, D10, D11, D12, D2, D3, D4, D5, D6, D7, D8, D9: footprint (none) -> Diode_THT:D_DO-41_SOD81_P3.81mm_Vertical_AnodeUp
- J2: footprint (none) -> Connector_PinHeader_2.54mm:PinHeader_1x06_P2.54mm_Vertical
- SW1, SW10, SW11, SW12, SW2, SW3, SW4, SW5, SW6, SW7, SW8, SW9: footprint (none) -> PCM_Switch_Keyboard_Cherry_MX:SW_Cherry_MX_PCB
- U1: footprint ADAFRUIT_QT_PY:MODULE_ADAFRUIT_QT_PY -> qtpy:MODULE_ADAFRUIT_QT_PY
Connections:
- net col0: now also U1.5 (D4/SDA); no longer U1.9 (A8/D8/SCK)
- net col1: now also U1.6 (D5/SCL); no longer U1.10 (A9/D9/MISO)
- net col2: now also U1.7 (A6/D6/TX); no longer U1.11 (A10/D10/MOSI)
- net ext0: now also J2.4 (Pin_4), U1.11 (A10/D10/MOSI); no longer J2.1 (Pin_1), U1.5 (D4/SDA)
- net ext1: now also J2.3 (Pin_3), U1.10 (A9/D9/MISO); no longer J2.2 (Pin_2), U1.6 (D5/SCL)
- net ext2: now also J2.2 (Pin_2), U1.9 (A8/D8/SCK); no longer J2.3 (Pin_3), U1.7 (A6/D6/TX)
- net ext3: now also J2.1 (Pin_1); no longer J2.4 (Pin_4)
- net row0: now also U1.4 (A3/D3); no longer U1.1 (A0/D0/DAC)
- net row1: now also U1.3 (A2/D2); no longer U1.2 (A1/D1)
- net row2: now also U1.2 (A1/D1); no longer U1.3 (A2/D2)
- net row3: now also U1.1 (A0/D0/DAC); no longer U1.4 (A3/D3)
Changed lines of the file:
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@@
 		)
 	)
-	(label "row2"
+	(label "row1"
 		(at 39.37 71.12 0)
 		(fields_autoplaced yes)
@@
 		)
 	)
-	(label "row0"
+	(label "row3"
 		(at 39.37 66.04 0)
 		(fields_autoplaced yes)
@@
 		)
 	)
-	(label "ext0"
+	(label "ext3"
 		(at 69.85 120.65 0)
 		(fields_autoplaced yes)
@@
 		)
 	)
-	(label "ext0"
+	(label "col0"
 		(at 39.37 76.2 0)
 		(fields_autoplaced yes)
@@
 		)
 	)
-	(label "col1"
+	(label "ext1"
 		(at 90.17 73.66 0)
 		(fields_autoplaced yes)
@@
 		)
 	)
-	(label "ext1"
+	(label "ext2"
 		(at 69.85 118.11 0)
 		(fields_autoplaced yes)
@@
 		)
 	)
-	(label "col2"
+	(label "ext0"
 		(at 90.17 76.2 0)
 		(fields_autoplaced yes)
@@
 		)
 	)
-	(label "col0"
+	(label "ext2"
 		(at 90.17 71.12 0)
 		(fields_autoplaced yes)
@@
 		)
 	)
-	(label "ext1"
+	(label "col1"
 		(at 39.37 78.74 0)
 		(fields_autoplaced yes)
@@
 		)
 	)
-	(label "ext2"
+	(label "col2"
 		(at 90.17 66.04 0)
 		(fields_autoplaced yes)
@@
 		)
 	)
-	(label "ext2"
+	(label "ext1"
 		(at 69.85 115.57 0)
 		(fields_autoplaced yes)
@@
 		)
 	)
-	(label "ext3"
+	(label "ext0"
 		(at 69.85 113.03 0)
 		(fields_autoplaced yes)
@@
 		)
 	)
-	(label "row1"
+	(label "row2"
 		(at 39.37 68.58 0)
 		(fields_autoplaced yes)
@@
 		)
 	)
-	(label "row3"
+	(label "row0"
 		(at 39.37 73.66 0)
 		(fields_autoplaced yes)
@@
 			)
 		)
-		(property "Footprint" ""
+		(property "Footprint" "Diode_THT:D_DO-41_SOD81_P3.81mm_Vertical_AnodeUp"
 			(at 179.07 109.22 0)
 			(effects
@@
 			)
 		)
-		(property "Footprint" ""
+		(property "Footprint" "PCM_Switch_Keyboard_Cherry_MX:SW_Cherry_MX_PCB"
 			(at 161.29 62.23 0)
 			(effects
@@
 			)
 		)
-		(property "Footprint" ""
+		(property "Footprint" "PCM_Switch_Keyboard_Cherry_MX:SW_Cherry_MX_PCB"
 			(at 138.43 100.33 0)
 			(effects
@@
 			)
 		)
-		(property "Footprint" ""
+		(property "Footprint" "Diode_THT:D_DO-41_SOD81_P3.81mm_Vertical_AnodeUp"
 			(at 179.07 71.12 0)
 			(effects
@@
 			)
 		)
-		(property "Footprint" ""
+		(property "Footprint" "PCM_Switch_Keyboard_Cherry_MX:SW_Cherry_MX_PCB"
 			(at 184.15 43.18 0)
 			(effects
@@
 			)
 		)
-		(property "Footprint" ""
+		(property "Footprint" "PCM_Switch_Keyboard_Cherry_MX:SW_Cherry_MX_PCB"
 			(at 138.43 43.18 0)
 			(effects
@@
 			)
 		)
-		(property "Footprint" ""
+		(property "Footprint" "PCM_Switch_Keyboard_Cherry_MX:SW_Cherry_MX_PCB"
 			(at 184.15 100.33 0)
 			(effects
@@
 			)
 		)
-		(property "Footprint" ""
+		(property "Footprint" "PCM_Switch_Keyboard_Cherry_MX:SW_Cherry_MX_PCB"
 			(at 138.43 62.23 0)
 			(effects
@@
 			)
 		)
-		(property "Footprint" "ADAFRUIT_QT_PY:MODULE_ADAFRUIT_QT_PY"
+		(property "Footprint" "qtpy:MODULE_ADAFRUIT_QT_PY"
 			(at 67.31 71.12 0)
 			(effects
@@
 			)
 		)
-		(property "Footprint" ""
+		(property "Footprint" "Diode_THT:D_DO-41_SOD81_P3.81mm_Vertical_AnodeUp"
 			(at 133.35 109.22 0)
 			(effects
@@
 			)
 		)
-		(property "Footprint" ""
+		(property "Footprint" "PCM_Switch_Keyboard_Cherry_MX:SW_Cherry_MX_PCB"
 			(at 161.29 81.28 0)
 			(effects
@@
 			)
 		)
-		(property "Footprint" ""
+		(property "Footprint" "Connector_PinHeader_2.54mm:PinHeader_1x06_P2.54mm_Vertical"
 			(at 64.77 115.57 0)
 			(effects
@@
 			)
 		)
-		(property "Footprint" ""
+		(property "Footprint" "Diode_THT:D_DO-41_SOD81_P3.81mm_Vertical_AnodeUp"
 			(at 133.35 71.12 0)
 			(effects
@@
 			)
 		)
-		(property "Footprint" ""
+		(property "Footprint" "PCM_Switch_Keyboard_Cherry_MX:SW_Cherry_MX_PCB"
 			(at 184.15 81.28 0)
 			(effects
@@
 			)
 		)
-		(property "Footprint" ""
+		(property "Footprint" "PCM_Switch_Keyboard_Cherry_MX:SW_Cherry_MX_PCB"
 			(at 184.15 62.23 0)
 			(effects
@@
 			)
 		)
-		(property "Footprint" ""
+		(property "Footprint" "Diode_THT:D_DO-41_SOD81_P3.81mm_Vertical_AnodeUp"
 			(at 156.21 52.07 0)
 			(effects
@@
 			)
 		)
-		(property "Footprint" ""
+		(property "Footprint" "Diode_THT:D_DO-41_SOD81_P3.81mm_Vertical_AnodeUp"
 			(at 179.07 52.07 0)
 			(effects
@@
 			)
 		)
-		(property "Footprint" ""
+		(property "Footprint" "PCM_Switch_Keyboard_Cherry_MX:SW_Cherry_MX_PCB"
 			(at 138.43 81.28 0)
 			(effects
@@
 			)
 		)
-		(property "Footprint" ""
+		(property "Footprint" "Diode_THT:D_DO-41_SOD81_P3.81mm_Vertical_AnodeUp"
 			(at 133.35 90.17 0)
 			(effects
@@
 			)
 		)
-		(property "Footprint" ""
+		(property "Footprint" "Diode_THT:D_DO-41_SOD81_P3.81mm_Vertical_AnodeUp"
 			(at 156.21 90.17 0)
 			(effects
@@
 			)
 		)
-		(property "Footprint" ""
+		(property "Footprint" "Diode_THT:D_DO-41_SOD81_P3.81mm_Vertical_AnodeUp"
 			(at 156.21 109.22 0)
 			(effects
@@
 			)
 		)
-		(property "Footprint" ""
+		(property "Footprint" "Diode_THT:D_DO-41_SOD81_P3.81mm_Vertical_AnodeUp"
 			(at 179.07 90.17 0)
 			(effects
@@
 			)
 		)
-		(property "Footprint" ""
+		(property "Footprint" "Diode_THT:D_DO-41_SOD81_P3.81mm_Vertical_AnodeUp"
 			(at 156.21 71.12 0)
 			(effects
@@
 			)
 		)
-		(property "Footprint" ""
+		(property "Footprint" "PCM_Switch_Keyboard_Cherry_MX:SW_Cherry_MX_PCB"
 			(at 161.29 100.33 0)
 			(effects
@@
 			)
 		)
-		(property "Footprint" ""
+		(property "Footprint" "PCM_Switch_Keyboard_Cherry_MX:SW_Cherry_MX_PCB"
 			(at 161.29 43.18 0)
 			(effects
@@
 			)
 		)
-		(property "Footprint" ""
+		(property "Footprint" "Diode_THT:D_DO-41_SOD81_P3.81mm_Vertical_AnodeUp"
 			(at 133.35 52.07 0)
 			(effects

Commit message: Better pcb layout
Parts:
- D1, D10, D11, D12, D2, D3, D4, D5, D6, D7, D8, D9: footprint Diode_THT:D_DO-41_SOD81_P3.81mm_Vertical_AnodeUp -> Diode_SMD:D_1206_3216Metric_Pad1.42x1.75mm_HandSolder
- SW1, SW10, SW11, SW12, SW2, SW3, SW4, SW5, SW6, SW7, SW8, SW9: footprint PCM_Switch_Keyboard_Cherry_MX:SW_Cherry_MX_PCB -> mx_solderable:MX-Solderable-1U
Connections:
- net col0: now also U1.7 (A6/D6/TX); no longer U1.5 (D4/SDA)
- net col2: now also U1.5 (D4/SDA); no longer U1.7 (A6/D6/TX)
Changed lines of the file:
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@@
 		)
 	)
-	(label "col0"
+	(label "col2"
 		(at 39.37 76.2 0)
 		(fields_autoplaced yes)
@@
 		)
 	)
-	(label "col2"
+	(label "col0"
 		(at 90.17 66.04 0)
 		(fields_autoplaced yes)
@@
 			)
 		)
-		(property "Footprint" "Diode_THT:D_DO-41_SOD81_P3.81mm_Vertical_AnodeUp"
+		(property "Footprint" "Diode_SMD:D_1206_3216Metric_Pad1.42x1.75mm_HandSolder"
 			(at 179.07 109.22 0)
 			(effects
@@
 			)
 		)
-		(property "Footprint" "PCM_Switch_Keyboard_Cherry_MX:SW_Cherry_MX_PCB"
+		(property "Footprint" "mx_solderable:MX-Solderable-1U"
 			(at 161.29 62.23 0)
 			(effects
@@
 			)
 		)
-		(property "Footprint" "PCM_Switch_Keyboard_Cherry_MX:SW_Cherry_MX_PCB"
+		(property "Footprint" "mx_solderable:MX-Solderable-1U"
 			(at 138.43 100.33 0)
 			(effects
@@
 			)
 		)
-		(property "Footprint" "Diode_THT:D_DO-41_SOD81_P3.81mm_Vertical_AnodeUp"
+		(property "Footprint" "Diode_SMD:D_1206_3216Metric_Pad1.42x1.75mm_HandSolder"
 			(at 179.07 71.12 0)
 			(effects
@@
 			)
 		)
-		(property "Footprint" "PCM_Switch_Keyboard_Cherry_MX:SW_Cherry_MX_PCB"
+		(property "Footprint" "mx_solderable:MX-Solderable-1U"
 			(at 184.15 43.18 0)
 			(effects
@@
 			)
 		)
-		(property "Footprint" "PCM_Switch_Keyboard_Cherry_MX:SW_Cherry_MX_PCB"
+		(property "Footprint" "mx_solderable:MX-Solderable-1U"
 			(at 138.43 43.18 0)
 			(effects
@@
 			)
 		)
-		(property "Footprint" "PCM_Switch_Keyboard_Cherry_MX:SW_Cherry_MX_PCB"
+		(property "Footprint" "mx_solderable:MX-Solderable-1U"
 			(at 184.15 100.33 0)
 			(effects
@@
 			)
 		)
-		(property "Footprint" "PCM_Switch_Keyboard_Cherry_MX:SW_Cherry_MX_PCB"
+		(property "Footprint" "mx_solderable:MX-Solderable-1U"
 			(at 138.43 62.23 0)
 			(effects
@@
 			)
 		)
-		(property "Footprint" "Diode_THT:D_DO-41_SOD81_P3.81mm_Vertical_AnodeUp"
+		(property "Footprint" "Diode_SMD:D_1206_3216Metric_Pad1.42x1.75mm_HandSolder"
 			(at 133.35 109.22 0)
 			(effects
@@
 			)
 		)
-		(property "Footprint" "PCM_Switch_Keyboard_Cherry_MX:SW_Cherry_MX_PCB"
+		(property "Footprint" "mx_solderable:MX-Solderable-1U"
 			(at 161.29 81.28 0)
 			(effects
@@
 			)
 		)
-		(property "Footprint" "Diode_THT:D_DO-41_SOD81_P3.81mm_Vertical_AnodeUp"
+		(property "Footprint" "Diode_SMD:D_1206_3216Metric_Pad1.42x1.75mm_HandSolder"
 			(at 133.35 71.12 0)
 			(effects
@@
 			)
 		)
-		(property "Footprint" "PCM_Switch_Keyboard_Cherry_MX:SW_Cherry_MX_PCB"
+		(property "Footprint" "mx_solderable:MX-Solderable-1U"
 			(at 184.15 81.28 0)
 			(effects
@@
 			)
 		)
-		(property "Footprint" "PCM_Switch_Keyboard_Cherry_MX:SW_Cherry_MX_PCB"
+		(property "Footprint" "mx_solderable:MX-Solderable-1U"
 			(at 184.15 62.23 0)
 			(effects
@@
 			)
 		)
-		(property "Footprint" "Diode_THT:D_DO-41_SOD81_P3.81mm_Vertical_AnodeUp"
+		(property "Footprint" "Diode_SMD:D_1206_3216Metric_Pad1.42x1.75mm_HandSolder"
 			(at 156.21 52.07 0)
 			(effects
@@
 			)
 		)
-		(property "Footprint" "Diode_THT:D_DO-41_SOD81_P3.81mm_Vertical_AnodeUp"
+		(property "Footprint" "Diode_SMD:D_1206_3216Metric_Pad1.42x1.75mm_HandSolder"
 			(at 179.07 52.07 0)
 			(effects
@@
 			)
 		)
-		(property "Footprint" "PCM_Switch_Keyboard_Cherry_MX:SW_Cherry_MX_PCB"
+		(property "Footprint" "mx_solderable:MX-Solderable-1U"
 			(at 138.43 81.28 0)
 			(effects
@@
 			)
 		)
-		(property "Footprint" "Diode_THT:D_DO-41_SOD81_P3.81mm_Vertical_AnodeUp"
+		(property "Footprint" "Diode_SMD:D_1206_3216Metric_Pad1.42x1.75mm_HandSolder"
 			(at 133.35 90.17 0)
 			(effects
@@
 			)
 		)
-		(property "Footprint" "Diode_THT:D_DO-41_SOD81_P3.81mm_Vertical_AnodeUp"
+		(property "Footprint" "Diode_SMD:D_1206_3216Metric_Pad1.42x1.75mm_HandSolder"
 			(at 156.21 90.17 0)
 			(effects
@@
 			)
 		)
-		(property "Footprint" "Diode_THT:D_DO-41_SOD81_P3.81mm_Vertical_AnodeUp"
+		(property "Footprint" "Diode_SMD:D_1206_3216Metric_Pad1.42x1.75mm_HandSolder"
 			(at 156.21 109.22 0)
 			(effects
@@
 			)
 		)
-		(property "Footprint" "Diode_THT:D_DO-41_SOD81_P3.81mm_Vertical_AnodeUp"
+		(property "Footprint" "Diode_SMD:D_1206_3216Metric_Pad1.42x1.75mm_HandSolder"
 			(at 179.07 90.17 0)
 			(effects
@@
 			)
 		)
-		(property "Footprint" "Diode_THT:D_DO-41_SOD81_P3.81mm_Vertical_AnodeUp"
+		(property "Footprint" "Diode_SMD:D_1206_3216Metric_Pad1.42x1.75mm_HandSolder"
 			(at 156.21 71.12 0)
 			(effects
@@
 			)
 		)
-		(property "Footprint" "PCM_Switch_Keyboard_Cherry_MX:SW_Cherry_MX_PCB"
+		(property "Footprint" "mx_solderable:MX-Solderable-1U"
 			(at 161.29 100.33 0)
 			(effects
@@
 			)
 		)
-		(property "Footprint" "PCM_Switch_Keyboard_Cherry_MX:SW_Cherry_MX_PCB"
+		(property "Footprint" "mx_solderable:MX-Solderable-1U"
 			(at 161.29 43.18 0)
 			(effects
@@
 			)
 		)
-		(property "Footprint" "Diode_THT:D_DO-41_SOD81_P3.81mm_Vertical_AnodeUp"
+		(property "Footprint" "Diode_SMD:D_1206_3216Metric_Pad1.42x1.75mm_HandSolder"
 			(at 133.35 52.07 0)
 			(effects

Commit message: Initial prototype pcb
Connections:
- net col1: now also U1.10 (A9/D9/MISO); no longer U1.6 (D5/SCL)
- net col2: now also U1.11 (A10/D10/MOSI); no longer U1.5 (D4/SDA)
- net ext0: now also U1.5 (D4/SDA); no longer U1.11 (A10/D10/MOSI)
- net ext1: now also U1.6 (D5/SCL); no longer U1.10 (A9/D9/MISO)
Changed lines of the file:
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@@
+		)
+	)
+	(label "ext1"
+		(at 39.37 78.74 0)
+		(fields_autoplaced yes)
+		(effects
+			(font
+				(size 1.27 1.27)
+			)
+			(justify left bottom)
+		)
+	)
+	(label "col2"
+		(at 90.17 76.2 0)
+		(fields_autoplaced yes)
+		(effects
+			(font
+				(size 1.27 1.27)
+			)
+			(justify left bottom)
 		)
 	)
@@
 		)
 	)
-	(label "col2"
-		(at 39.37 76.2 0)
+	(label "col1"
+		(at 90.17 73.66 0)
 		(fields_autoplaced yes)
 		(effects
@@
 		)
 	)
-	(label "ext1"
-		(at 90.17 73.66 0)
-		(fields_autoplaced yes)
-		(effects
-			(font
-				(size 1.27 1.27)
-			)
-			(justify left bottom)
-		)
-	)
 	(label "ext2"
 		(at 69.85 118.11 0)
@@
 		)
 	)
-	(label "ext0"
-		(at 90.17 76.2 0)
-		(fields_autoplaced yes)
-		(effects
-			(font
-				(size 1.27 1.27)
-			)
-			(justify left bottom)
-		)
-	)
 	(label "col1"
 		(at 166.37 31.75 0)
@@
 	(label "ext2"
 		(at 90.17 71.12 0)
-		(fields_autoplaced yes)
-		(effects
-			(font
-				(size 1.27 1.27)
-			)
-			(justify left bottom)
-		)
-	)
-	(label "col1"
-		(at 39.37 78.74 0)
 		(fields_autoplaced yes)
 		(effects
@@
 		(fields_autoplaced yes)
 		(effects
+			(font
+				(size 1.27 1.27)
+			)
+			(justify left bottom)
+		)
+	)
+	(label "ext0"
+		(at 39.37 76.2 0)
+		(fields_autoplaced yes)
+		(effects
